File: PCB/Rev2/CustomPCB.kicad_pcb (KiCad board)
At the start: 2 copper layers, 41.4 x 107.3 mm, 29 parts, among them J1 Conn_01x06, J2 Conn_01x02, J3 Conn_01x03, Q1 AO3401A, SW1 RotaryEncoder, U1 PMW3610, U2 TLV74318PDBVR, U3 SuperMini nRF52840

Commit message: Update Rev2 and documentation
Parts:
- removed Q1: AO3401A, Package_TO_SOT_SMD:SOT-23
- removed R2: 10k, Resistor_SMD:R_0603_1608Metric
- added C11: 1uF, Capacitor_SMD:C_0603_1608Metric, F.Cu at (202.7, 96.3)
- added C12: 100nF, Capacitor_SMD:C_0603_1608Metric, F.Cu at (200.2, 90.4)
- added U4: TPS22917DBV, Package_TO_SOT_SMD:SOT-23-6, F.Cu at (203.7, 91.5)
Connections:
- U3 pad 22: GATE -> LED_CTRL
Routing:
- net GATE: track 35.7 -> 0.00 mm, vias 2 -> 0
- net LED_CTRL: track 0.00 -> 33.5 mm, vias 0 -> 2
- net LED_VCC: track 37.0 -> 41.1 mm
- net BAT+: track 12.7 -> 10.6 mm
